File: IC- Henrique Teixeira (nao acabada)/Communication-Board-main/communication_board/communication_board.kicad_sch (KiCad schematic)
At the start: 60 parts, among them J1 USB_IN, J10 B4B-XH-A, J11 B4B-XH-A, J12 XT60-M, J13 B4B-XH-A, J14 B4B-XH-A, J15 B4B-XH-A, J16 B4B-XH-A, J17 B4B-XH-A, J18 IMU, J2 IMU, J3 MINI_FUSE, J4 Motors, J5 XT60-M, J6 XT60-M, J7 B4B-XH-A, J8 B4B-XH-A, J9 B4B-XH-A, SW1 SW_DPST_x2, U1 FE1.1s, U2 FT232RL, U3 FT232RL, U4 MAX485E, Y1 Crystal

Commit message: Projeto do teclado mecanico split
Connections:
- net GND: now also J10.1, J11.1, J12.N (NEG), J13.1, J14.1, J15.1, J16.1, J17.1, J5.N (NEG), J6.N (NEG), J7.1, J8.1, J9.1; no longer A1.29 (GND), J18.7 (Pin_7)
- net GNDREF: now also A1.29 (GND), J18.7 (Pin_7); no longer J10.1, J11.1, J12.N (NEG), J13.1, J14.1, J15.1, J16.1, J17.1, J5.N (NEG), J6.N (NEG), J7.1, J8.1, J9.1
