File: IC- Henrique Teixeira (nao acabada)/Communication-Board-main/NEW_Communication_Board.kicad_pcb (KiCad board)
At the start: 4 copper layers, 103.2 x 58.9 mm, 74 parts, among them J1 USB_IN, J2 IMU, J3 Mini Fuse Socket, J4 XM_conn, J5 HUB-3, J6 HUB-4, U1 FE1.1s, U2 FT232RL, U3 FT232RL, U4 MAX485E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

Commit message: V2 communication Board
Parts:
- removed C23: 0.1uF, Capacitor_SMD:C_1206_3216Metric
- removed C24: 10uF, Capacitor_SMD:C_1206_3216Metric
- removed U4: MAX485E, Package_SO:SOIC-8_3.9x4.9mm_P1.27mm
- added U8: ST485E, Package_SO:SOIC-8_3.9x4.9mm_P1.27mm, F.Cu at (118.8, 73.0)
- D10: value ST_TX -> ARDUINO_TX
- D11: value ST_RX -> ARDUINO_RX
Connections:
- C21 pad 1: USB_PWR -> GNDREF
- C21 pad 2: GNDREF -> USB_PWR
Routing:
- net USB_PWR: track 290.9 -> 284.8 mm, vias 7 -> 8
- net GNDREF: track 66.4 -> 65.0 mm, vias 49 -> 46
Other:
- board text removed: "C23"
- board text removed: "C24"
